File: Hardware/v1/DCDC.sch (KiCad schematic (older format))
At the start: 37 parts, among them J1 BAT_CONN, J2 EN_BAT_VIN, J3 USB_A_PWR_OUTPUT, Q1 DMN62D0UW-7, SW1 MCU_USB_POWER, U1 TPS54561DPRR, U2 MCP16311MS, U3 PDS760-13

Commit message: bah
Connections:
- net PWR_5V renamed +5V
Changed lines of the file:
@@
 $EndComp
 $Comp
-L power:GND #PWR05
+L power:GND #PWR08
 U 1 1 5D84EAB6
 P 2550 7400
-F 0 "#PWR05" H 2550 7150 50  0001 C CNN
+F 0 "#PWR08" H 2550 7150 50  0001 C CNN
 F 1 "GND" H 2555 7227 50  0000 C CNN
 F 2 "" H 2550 7400 50  0001 C CNN
@@
 $EndComp
 $Comp
-L power:VCC #PWR08
+L power:VCC #PWR012
 U 1 1 5DA67011
 P 4550 5750
-F 0 "#PWR08" H 4550 5600 50  0001 C CNN
+F 0 "#PWR012" H 4550 5600 50  0001 C CNN
 F 1 "VCC" H 4567 5923 50  0000 C CNN
 F 2 "" H 4550 5750 50  0001 C CNN
@@
 Connection ~ 2100 1050
 $Comp
-L power:GND #PWR06
+L power:GND #PWR09
 U 1 1 5D9E9F0B
 P 2800 3250
-F 0 "#PWR06" H 2800 3000 50  0001 C CNN
+F 0 "#PWR09" H 2800 3000 50  0001 C CNN
 F 1 "GND" H 2805 3077 50  0000 C CNN
 F 2 "" H 2800 3250 50  0001 C CNN
@@
 	2800 3050 2800 3150
 $Comp
-L power:GND #PWR07
+L power:GND #PWR010
 U 1 1 5D9EA2F0
 P 4300 2350
-F 0 "#PWR07" H 4300 2100 50  0001 C CNN
+F 0 "#PWR010" H 4300 2100 50  0001 C CNN
 F 1 "GND" H 4305 2177 50  0000 C CNN
 F 2 "" H 4300 2350 50  0001 C CNN
@@
 $EndComp
 $Comp
-L power:GND #PWR010
+L power:GND #PWR014
 U 1 1 5DA4D56B
 P 5400 4150
-F 0 "#PWR010" H 5400 3900 50  0001 C CNN
+F 0 "#PWR014" H 5400 3900 50  0001 C CNN
 F 1 "GND" H 5405 3977 50  0000 C CNN
 F 2 "" H 5400 4150 50  0001 C CNN
@@
 Wire Wire Line
 	5400 4050 5400 4150
-Text GLabel 6800 3400 2    50   Input ~ 0
-PWR_5V
 Wire Wire Line
 	5750 3750 5750 3400
@@
 $EndComp
 $Comp
-L power:GND #PWR011
+L power:GND #PWR015
 U 1 1 5DAA1187
 P 6400 4650
-F 0 "#PWR011" H 6400 4400 50  0001 C CNN
+F 0 "#PWR015" H 6400 4400 50  0001 C CNN
 F 1 "GND" H 6405 4477 50  0000 C CNN
 F 2 "" H 6400 4650 50  0001 C CNN
@@
 $EndComp
 NoConn ~ 6300 5600
-Text GLabel 1800 5950 0    50   Input ~ 0
-PWR_5V
-Text GLabel 6950 5700 2    50   Input ~ 0
-PWR_5V
-Wire Wire Line
-	6700 5700 6950 5700
 Wire Wire Line
 	4550 3400 4550 3300
@@
 Wire Wire Line
 	4000 2600 4400 2600
-Text GLabel 1550 3600 2    50   Input ~ 0
-PWR_5V
 $Comp
 L favorites:TPS54561DPRR U1
@@
 Wire Wire Line
 	1850 1850 2100 1850
-$Comp
-L power:PWR_FLAG #FLG03
-U 1 1 5DB2DE1C
-P 6650 3400
-F 0 "#FLG03" H 6650 3475 50  0001 C CNN
-F 1 "PWR_FLAG" H 6650 3573 50  0000 C CNN
-F 2 "" H 6650 3400 50  0001 C CNN
-F 3 "~" H 6650 3400 50  0001 C CNN
-	1    6650 3400
-	1    0    0    -1
-$EndComp
-Connection ~ 6650 3400
-Wire Wire Line
-	6650 3400 6800 3400
 Text GLabel 2100 2100 0    50   Input ~ 0
 BAT_VIN
@@
 	6400 3900 6400 3400
 Connection ~ 6400 3400
-Wire Wire Line
-	6400 3400 6650 3400
 Text Notes 2050 750  0    50   ~ 0
 Kanske behövs sådär 1206 capar
@@
 BAT_VIN
 $Comp
-L power:GND #PWR09
+L power:GND #PWR013
 U 1 1 5DA40EC4
 P 4850 2150
-F 0 "#PWR09" H 4850 1900 50  0001 C CNN
+F 0 "#PWR013" H 4850 1900 50  0001 C CNN
 F 1 "GND" H 4855 1977 50  0000 C CNN
 F 2 "" H 4850 2150 50  0001 C CNN
@@
 Text Notes 1900 1250 0    50   ~ 0
 12061C225KAT2A CAP CER 2.2UF 100V X7R 1206\nC3216X7S2A225K160AB CAP CER 2.2UF 100V X7S 1206\n
-Text GLabel 4600 1300 0    50   Input ~ 0
-PWR_5V
 $Comp
 L favorites:3PIN_DIODE U3
@@
 Wire Wire Line
 	5000 1100 5000 1050
-Wire Wire Line
-	4700 1300 4600 1300
 $Comp
 L Device:C_Small C16
@@
 EndData
 $EndBitmap
+$Comp
+L power:+5V #PWR011
+U 1 1 5E170600
+P 4450 1250
+F 0 "#PWR011" H 4450 1100 50  0001 C CNN
+F 1 "+5V" H 4465 1423 50  0000 C CNN
+F 2 "" H 4450 1250 50  0001 C CNN
+F 3 "" H 4450 1250 50  0001 C CNN
+	1    4450 1250
+	1    0    0    -1
+$EndComp
+Wire Wire Line
+	4450 1300 4450 1250
+Wire Wire Line
+	4450 1300 4700 1300
+$Comp
+L power:+5V #PWR05
+U 1 1 5E170A1F
+P 1800 3550
+F 0 "#PWR05" H 1800 3400 50  0001 C CNN
+F 1 "+5V" H 1815 3723 50  0000 C CNN
+F 2 "" H 1800 3550 50  0001 C CNN
+F 3 "" H 1800 3550 50  0001 C CNN
+	1    1800 3550
+	1    0    0    -1
+$EndComp
+Wire Wire Line
+	1550 3600 1800 3600
+Wire Wire Line
+	1800 3600 1800 3550
+$Comp
+L power:+5V #PWR06
+U 1 1 5E1721C9
+P 1800 5950
+F 0 "#PWR06" H 1800 5800 50  0001 C CNN
+F 1 "+5V" H 1815 6123 50  0000 C CNN
+F 2 "" H 1800 5950 50  0001 C CNN
+F 3 "" H 1800 5950 50  0001 C CNN
+	1    1800 5950
+	1    0    0    -1
+$EndComp
+$Comp
+L power:+5V #PWR017
+U 1 1 5E172D88
+P 7050 5600
+F 0 "#PWR017" H 7050 5450 50  0001 C CNN
+F 1 "+5V" H 7065 5773 50  0000 C CNN
+F 2 "" H 7050 5600 50  0001 C CNN
+F 3 "" H 7050 5600 50  0001 C CNN
+	1    7050 5600
+	1    0    0    -1
+$EndComp
+Wire Wire Line
+	7050 5700 7050 5600
+Wire Wire Line
+	6700 5700 7050 5700
+$Comp
+L power:+5V #PWR07
+U 1 1 5E1743A9
+P 1950 5450
+F 0 "#PWR07" H 1950 5300 50  0001 C CNN
+F 1 "+5V" H 1965 5623 50  0000 C CNN
+F 2 "" H 1950 5450 50  0001 C CNN
+F 3 "" H 1950 5450 50  0001 C CNN
+	1    1950 5450
+	1    0    0    -1
+$EndComp
+$Comp
+L power:PWR_FLAG #FLG03
+U 1 1 5E174777
+P 1950 5450
+F 0 "#FLG03" H 1950 5525 50  0001 C CNN
+F 1 "PWR_FLAG" V 1950 5578 50  0000 L CNN
+F 2 "" H 1950 5450 50  0001 C CNN
+F 3 "~" H 1950 5450 50  0001 C CNN
+	1    1950 5450
+	0    1    1    0
+$EndComp
+Wire Wire Line
+	6400 3400 6800 3400
+$Comp
+L power:+5V #PWR016
+U 1 1 5E176400
+P 6800 3400
+F 0 "#PWR016" H 6800 3250 50  0001 C CNN
+F 1 "+5V" H 6815 3573 50  0000 C CNN
+F 2 "" H 6800 3400 50  0001 C CNN
+F 3 "" H 6800 3400 50  0001 C CNN
+	1    6800 3400
+	1    0    0    -1
+$EndComp
 $EndSCHEMATC
