File: Hardware/v1/v1.kicad_pcb (KiCad board)
At the start: 4 copper layers, 81 x 50 mm, 93 parts, among them J1 BAT_CONN, J10 DACS, J11 SERV_0, J12 SERV_1, J13 SERV_2, J14 SERV_3, J15 SERV_4, J16 SERV_5, J17 SERV_6, J18 SERV_7, J19 CAN, J2 EN_BAT_VIN, J20 USB_B_Mini, J3 USB_A_PWR_OUTPUT, J4 GPIO1, J5 GPIO2, J6 GPIO3, P1 SWD, Q1 DMN62D0UW-7, SW1 MCU_USB_POWER, SW2 BOOT0, U1 TPS54561DPRR, U2 MCP16311MS, U3 PDS760-13, U4 BMI160, U5 STM32F405RGTx, U6 TJA1051TK-3, Y1 8Mhz

Commit message: added some text to silks
Other:
- board text added: "CANH"
- board text added: "CANL"
